Commit message: urdf/움직임 고도화

File: Assets/Robots/FactoryAMR/factory_amr.urdf (robot description, URDF)
Before this commit: robot factory_amr, 12 links, 11 joints
Links:
- added link front_left_steering, mass 0.5
- added link front_right_steering, mass 0.5
- link base_link: geometry collision box size=0.8 0.5 0.25; visual box size=0.8 0.5 0.25
Joints:
- added joint front_left_steering_joint: type revolute, parent base_link, child front_left_steering, origin xyz=0.3 0.325 0 rpy=0 0 0, axis 0 0 1, limit lower=-0.6 upper=0.6 effort=100 velocity=2
- added joint front_right_steering_joint: type revolute, parent base_link, child front_right_steering, origin xyz=0.3 -0.325 0 rpy=0 0 0, axis 0 0 1, limit lower=-0.6 upper=0.6 effort=100 velocity=2
- joint front_left_wheel_joint: origin xyz=0.3 0.325 0 rpy=0 0 0 -> xyz=0 0 0 rpy=0 0 0; parent base_link -> front_left_steering
- joint front_right_wheel_joint: origin xyz=0.3 -0.325 0 rpy=0 0 0 -> xyz=0 0 0 rpy=0 0 0; parent base_link -> front_right_steering

Commit message: 상판 크기 조절 및 애커만 조향 로직 수정

File: Assets/Robots/FactoryAMR/factory_amr.urdf (robot description, URDF)
Before this commit: robot factory_amr, 14 links, 13 joints
Links:
- link top_plate: geometry collision box size=0.75 0.45 0.02; visual box size=0.75 0.45 0.02

Commit message: 유니티-ROS 연결을 통해 카메라 기능 구현

File: Assets/Robots/FactoryAMR/factory_amr.urdf (robot description, URDF)
Before this commit: robot factory_amr, 14 links, 13 joints
Joints:
- joint camera_joint: origin xyz=0.02 0 0.2 rpy=0 0.2 0 -> xyz=0.02 0 0.2 rpy=0 0 0

Commit message: URDF(초음파, 레이더, 라이더, 카메라 센서 추가 및 수정), 센서 기능 활성화 및 ROS 토픽 기능 추가

File: Assets/Robots/FactoryAMR/factory_amr.urdf (robot description, URDF)
Before this commit: robot factory_amr, 14 links, 13 joints
Links:
- added link lidar_mount, mass 0.3; collision cylinder length=0.15 radius=0.02; visual cylinder length=0.15 radius=0.02
- added link radar_front_link, mass 0.2; collision box size=0.03 0.1 0.03; visual box size=0.03 0.1 0.03
- added link radar_rear_link, mass 0.2; collision box size=0.03 0.1 0.03; visual box size=0.03 0.1 0.03
- added link ultrasonic_fl_link, mass 0.05; collision cylinder length=0.02 radius=0.015; visual cylinder length=0.02 radius=0.015
- added link ultrasonic_fr_link, mass 0.05; collision cylinder length=0.02 radius=0.015; visual cylinder length=0.02 radius=0.015
- added link ultrasonic_rl_link, mass 0.05; collision cylinder length=0.02 radius=0.015; visual cylinder length=0.02 radius=0.015
- added link ultrasonic_rr_link, mass 0.05; collision cylinder length=0.02 radius=0.015; visual cylinder length=0.02 radius=0.015
- link camera_mount: mass 0.2 -> 0.1; geometry collision cylinder length=0.07 radius=0.012; visual cylinder length=0.07 radius=0.012
- link lidar_link: mass 0.5 -> 0.3; geometry collision cylinder length=0.05 radius=0.04; visual cylinder length=0.05 radius=0.04
Joints:
- added joint lidar_mount_joint: type fixed, parent top_plate, child lidar_mount, origin xyz=0 0 0.01 rpy=0 0 0
- added joint radar_front_joint: type fixed, parent base_link, child radar_front_link, origin xyz=0.41 0 0.1 rpy=0 0 0
- added joint radar_rear_joint: type fixed, parent base_link, child radar_rear_link, origin xyz=-0.41 0 0.1 rpy=0 0 3.1416
- added joint ultrasonic_fl_joint: type fixed, parent base_link, child ultrasonic_fl_link, origin xyz=0.38 0.23 0.1 rpy=0 0 0.7854
- added joint ultrasonic_fr_joint: type fixed, parent base_link, child ultrasonic_fr_link, origin xyz=0.38 -0.23 0.1 rpy=0 0 -0.7854
- added joint ultrasonic_rl_joint: type fixed, parent base_link, child ultrasonic_rl_link, origin xyz=-0.38 0.23 0.1 rpy=0 0 2.3562
- added joint ultrasonic_rr_joint: type fixed, parent base_link, child ultrasonic_rr_link, origin xyz=-0.38 -0.23 0.1 rpy=0 0 -2.3562
- joint camera_joint: origin xyz=0.02 0 0.2 rpy=0 0 0 -> xyz=0 0 0.09 rpy=0 0 0
- joint camera_mount_joint: origin xyz=-0.2 0 0.01 rpy=0 0 0 -> xyz=0.35 0 0.25 rpy=0 0 0; parent top_plate -> base_link
- joint imu_joint: origin xyz=0 0 0.25 rpy=0 0 0 -> xyz=0 0 0.26 rpy=0 0 0
- joint lidar_joint: origin xyz=0.3 0 0.01 rpy=0 0 0 -> xyz=0 0 0.175 rpy=0 0 0; parent top_plate -> lidar_mount

Commit message: 강화학습을 위한 차선 인식 기능 구현 중

File: Assets/Robots/FactoryAMR/factory_amr.urdf (robot description, URDF)
Before this commit: robot factory_amr, 21 links, 20 joints
Links:
- link camera_mount: geometry collision cylinder length=0.7 radius=0.012; visual cylinder length=0.7 radius=0.012
Joints:
- joint camera_joint: origin xyz=0 0 0.09 rpy=0 0 0 -> xyz=0 0 0.72 rpy=0 0 0

Commit message: KajamansRoads 에셋 다운 및 학습 데이터(front_image + speed) 변경 및 그에 따른 학습 데이터 수집 코드 수정(다양한 이미지 형식  + 회귀 방식(조향각, 가속도) 수집) 및  차량 구동 방식 코드 수정

File: Assets/Robots/FactoryAMR/factory_amr.urdf (robot description, URDF)
Before this commit: robot factory_amr, 21 links, 20 joints
Links:
- link base_link: geometry collision box size=0.8 0.5 0.4; visual box size=0.8 0.5 0.4
- link camera_mount: geometry collision cylinder length=0.5 radius=0.012; visual cylinder length=0.5 radius=0.012
Joints:
- joint camera_joint: origin xyz=0 0 0.72 rpy=0 0 0 -> xyz=0 0 0.52 rpy=0 0 0
- joint camera_mount_joint: origin xyz=0.35 0 0.25 rpy=0 0 0 -> xyz=0.35 0 0.40 rpy=0 0 0
- joint front_left_steering_joint: limit lower=-0.6 upper=0.6 effort=100 velocity=2 -> lower=-0.6 upper=0.6 effort=200 velocity=3
- joint front_left_wheel_joint: limit effort=10 velocity=20 -> effort=30 velocity=60
- joint front_right_steering_joint: limit lower=-0.6 upper=0.6 effort=100 velocity=2 -> lower=-0.6 upper=0.6 effort=200 velocity=3
- joint front_right_wheel_joint: limit effort=10 velocity=20 -> effort=30 velocity=60
- joint imu_joint: origin xyz=0 0 0.26 rpy=0 0 0 -> xyz=0 0 0.41 rpy=0 0 0
- joint rear_left_wheel_joint: limit effort=10 velocity=20 -> effort=30 velocity=60
- joint rear_right_wheel_joint: limit effort=10 velocity=20 -> effort=30 velocity=60
- joint top_plate_joint: origin xyz=0 0 0.26 rpy=0 0 0 -> xyz=0 0 0.41 rpy=0 0 0

Commit message: 맵 수정 및 urdf 수정

File: Assets/Robots/FactoryAMR/factory_amr.urdf (robot description, URDF)
Before this commit: robot factory_amr, 21 links, 20 joints
Links:
- link camera_mount: geometry collision cylinder length=0.2 radius=0.012; visual cylinder length=0.2 radius=0.012
- link lidar_mount: geometry collision cylinder length=0.3 radius=0.02; visual cylinder length=0.3 radius=0.02
Joints:
- joint camera_joint: origin xyz=0 0 0.52 rpy=0 0 0 -> xyz=0 0 0.22 rpy=0 0 0
- joint lidar_joint: origin xyz=0 0 0.175 rpy=0 0 0 -> xyz=0 0 0.325 rpy=0 0 0

Commit message: 강화학습을 위한 센서 데이터 기능 고도화 및 urdf 수정

File: Assets/Robots/FactoryAMR/factory_amr.urdf (robot description, URDF)
Before this commit: robot factory_amr, 21 links, 20 joints
Links:
- added link ultrasonic_fc_link, mass 0.05; collision cylinder length=0.02 radius=0.015; visual cylinder length=0.02 radius=0.015
- added link ultrasonic_rc_link, mass 0.05; collision cylinder length=0.02 radius=0.015; visual cylinder length=0.02 radius=0.015
Joints:
- added joint ultrasonic_fc_joint: type fixed, parent base_link, child ultrasonic_fc_link, origin xyz=0.41 0 0.1 rpy=0 0 0
- added joint ultrasonic_rc_joint: type fixed, parent base_link, child ultrasonic_rc_link, origin xyz=-0.41 0 0.1 rpy=0 0 3.1416
