Commit message: refactor(unity): replace FactoryAMR with AutoCar setup
- add AutoCar setup editor script and train prefab assets
- migrate robot URDF and materials from FactoryAMR to AutoCar
- remove RootAMR_Test and obsolete FactoryAMR assets

File: Assets/Robots/AutoCar/AutoCar.urdf (robot description, URDF)
Before this commit: robot factory_amr, 23 links, 22 joints
Links:
- added link ultrasonic_sl_link, mass 0.05; collision cylinder length=0.02 radius=0.015; visual cylinder length=0.02 radius=0.015
- added link ultrasonic_sr_link, mass 0.05; collision cylinder length=0.02 radius=0.015; visual cylinder length=0.02 radius=0.015
Joints:
- added joint ultrasonic_sl_joint: type fixed, parent base_link, child ultrasonic_sl_link, origin xyz=0 0.23 0.1 rpy=0 0 1.5708
- added joint ultrasonic_sr_joint: type fixed, parent base_link, child ultrasonic_sr_link, origin xyz=0 -0.23 0.1 rpy=0 0 -1.5708
- joint ultrasonic_fc_joint: origin xyz=0.41 0 0.1 rpy=0 0 0 -> xyz=0.39 0 0.1 rpy=0 0 0
- joint ultrasonic_fl_joint: origin xyz=0.38 0.23 0.1 rpy=0 0 0.7854 -> xyz=0.36 0.21 0.1 rpy=0 0 0.7854
- joint ultrasonic_fr_joint: origin xyz=0.38 -0.23 0.1 rpy=0 0 -0.7854 -> xyz=0.36 -0.21 0.1 rpy=0 0 -0.7854
- joint ultrasonic_rc_joint: origin xyz=-0.41 0 0.1 rpy=0 0 3.1416 -> xyz=-0.39 0 0.1 rpy=0 0 3.1416
- joint ultrasonic_rl_joint: origin xyz=-0.38 0.23 0.1 rpy=0 0 2.3562 -> xyz=-0.36 0.21 0.1 rpy=0 0 2.3562
- joint ultrasonic_rr_joint: origin xyz=-0.38 -0.23 0.1 rpy=0 0 -2.3562 -> xyz=-0.36 -0.21 0.1 rpy=0 0 -2.3562
